File: SmarterWatch_KiCad/_autosave-Smarter Watch Stuff.kicad_pcb (KiCad board)
At the start: 4 copper layers, 39.5 x 39.5 mm, 72 parts, among them J3 CX70M-24P1, M1 Motor_DC, Q1 2N7002, Q2 2N7002, Q3 2N7002, Q4 2N7002, SW1 SW_SPST, SW2 SW_SPST, U1 MCP7940N-xSN, U10 MAX30102, U11 BMI160, U12 M24C64-WMN6TP, U2 TSL25911FN, U3 MCP73831-2-MC, U4 TCR2EE10, U5 ESP32-C6-MINI-1, U6 SHTC3, U7 TMP117xxDRV, U9 MIC5365-1.8YC5, Y1 Crystal

Commit message: Finished touting!
Finished routing.
Parts:
- moved C19 0.40 mm to (61.2, 79.3)
- moved C16 0.32 mm to (61.1, 77.1)
- moved R23 0.30 mm to (61.9, 79.1)
Routing:
- net GND: track 144.6 -> 233.9 mm, vias 10 -> 23
- net +3.3V: track 83.0 -> 98.8 mm, vias 6 -> 11
- net SCL: track 77.0 -> 91.4 mm, vias 6 -> 7
- net Net-(U10-VDD): track 2.92 -> 14.9 mm, vias 0 -> 2
- net Net-(U13-VREG): track 3.25 -> 11.2 mm
- net +3.3V_sensor: track 63.8 -> 66.2 mm, vias 6 -> 7
- net SDA: track 96.4 -> 96.6 mm, vias 4 -> 6
