File: SmarterWatch_KiCad/_autosave-Smarter Watch Stuff.kicad_pcb (KiCad board)
At the start: 4 copper layers, 39 x 39 mm, 111 parts, among them J5 CX70M-24P1, M1 Motor_DC, Q1 2N7002, Q2 2N7002, Q3 2N7002, Q4 2N7002, SW1 SW_SPST, SW2 SW_SPST, U1 MCP7940N-xSN, U10 MAX30102, U11 BMI160, U15 M24C64-WMN6TP, U16 IQS323001DNR, U17 MAX30205MTA+T, U2 TSL25911FN, U21 MMC5983MA, U24 AS3935-BQFT, U25 SGP40-D-R4, U26 NLA9306MU3TAG, U3 MCP73831-2-MC, U4 TCR2EE10, U5 ESP32-C6-MINI-1, U6 SHTC3, U7 TMP117xxDRV, U8 ST7735, U9 MIC5365-1.8YC5, Y1 Crystal

Commit message: upgrades people upgrades
Parts:
- removed C2, C3: 12 picoF, Capacitor_SMD:C_0402_1005Metric
- removed U1: MCP7940N-xSN, Package_SO:JEITA_SOIC-8_3.9x4.9mm_P1.27mm
- removed Y1: Crystal, Custom_Foot:XTAL_SC32S-7PF20PPM_EPS
- moved C6 87.4 mm to (74.2, 50.8)
- moved C16 83.7 mm to (101.3, 53.8), turned to 180 degrees
- moved C27 82.4 mm to (77.2, 76.8), turned to -90 degrees
- moved C17 80.6 mm to (104.5, 57.2)
- moved R34 79.8 mm to (77.2, 74.9), turned to -90 degrees
- moved C15 79.2 mm to (104.5, 54.7)
- moved R1 77.5 mm to (81.0, 52.3)
- moved C5 75.0 mm to (80.5, 62.3), turned to 180 degrees
- moved C21 18.1 mm to (168.9, 93.2)
- moved C14 1.65 mm to (81.1, 53.9), turned to -90 degrees
- moved R25 0.57 mm to (105.0, 52.9)
- moved C4 0.49 mm to (77.2, 78.6)
- moved U25 0.32 mm to (75.0, 74.7)
- moved U2 0.22 mm to (74.9, 77.5)
- moved R23 0.10 mm to (105.0, 58.6)
Routing:
- net GND: track 323.9 -> 347.2 mm, vias 12 -> 15
- net Net-(U16-VREG): track 0.00 -> 16.9 mm, vias 0 -> 3
- net Net-(U25-VDD): track 0.00 -> 8.05 mm, vias 0 -> 2
- net +3.3V: track 108.1 -> 115.6 mm
- net Net-(U16-RDY/MCLR): track 0.00 -> 2.06 mm
- net +5V: track 23.7 -> 25.0 mm
- net Net-(U3-PROG): track 0.00 -> 1.15 mm
- net +BATT: track 24.0 -> 25.0 mm
- net Net-(U16-CRX0/CTX0): track 2.83 -> 3.50 mm
- net CRX2: track 3.15 -> 2.60 mm
