File: SmarterWatch_KiCad/Lightning.kicad_sch (KiCad schematic)
At the start: 10 parts, among them U24 AS3935-BQFT

Commit message: Label Jumpers
Parts:
- U22, U23: footprint Custom_Foot:Jumper_NO -> (none)
Changed lines of the file:
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@@
 			)
 		)
-		(property "Footprint" "Custom_Foot:Jumper_NO"
+		(property "Footprint" ""
 			(at 93.98 100.33 0)
 			(effects
@@
 			)
 		)
-		(property "Footprint" "Custom_Foot:Jumper_NO"
+		(property "Footprint" ""
 			(at 93.98 92.71 0)
 			(effects
