File: SmarterWatch_KiCad/Lightning.kicad_sch (KiCad schematic)
At the start: 1 part, among them U19 AS3935-BQFT

Commit message: a bunch of light
Parts:
- added BT2: Battery_Cell, symbol Device:Battery_Cell
- added C23: CBAT, symbol Device:C
- added C24: 10UF, symbol Device:C
- added R31: R, symbol Device:R
Connections:
- net at U19.1 (ACG): now also C24.1
- net SCL: now reaches U19.11 (I2CL/SCL)
- net SCL: now also R31.2
- net GND: now reaches U19.12 (MISO)
- net GND: now also U19.4 (GND), U19.7 (EN_VREG), U19.8 (~{CS}), BT2.2 (-), C23.2, C24.2
- net SDA: now reaches U19.13 (I2CD/MOSI)
- net +3.3V: now reaches U19.5 (VDD)
- net +3.3V: now also U19.6 (VREG), BT2.1 (+), C23.1, R31.1
- no-connect marks 0 -> 1

Commit message: Final Lighning done just need values
Parts:
- added C25: C, symbol Device:C
- added L1: L, symbol Device:L
- added R32, R33: 10k, symbol Device:R
- added R34: R, symbol Device:R
- added U21, U22: ~, symbol Custom:OpenJumper
Connections:
- net +3.3V: now also U19.9 (SI), U21.2, U22.2
- net GND: now also U19.17 (EXP), U19.2 (INN), C25.1, L1.1, R32.2, R33.2, R34.1
- net at U19.15 (ADD0): now also R32.1, U22.1
- net at U19.16 (ADD1): now also R33.1, U21.1
- net at U19.3 (INP): now also C25.2, L1.2, R34.2

Commit message: order
Parts:
- removed BT2: Battery_Cell, symbol Device:Battery_Cell
Changed lines of the file:
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@@
 	(paper "A4")
-	(junction
-		(at 193.04 78.74)
-		(diameter 0)
-		(color 0 0 0 0)
-	)
 	(junction
 		(at 187.96 71.12)
@@
 	)
 	(junction
-		(at 193.04 71.12)
-		(diameter 0)
-		(color 0 0 0 0)
-	)
-	(junction
 		(at 177.8 74.93)
 		(diameter 0)
@@
 	(wire
 		(pts
-			(xy 193.04 71.12) (xy 195.58 71.12)
-		)
-		(stroke
-			(width 0)
-			(type default)
-		)
-	)
-	(wire
-		(pts
 			(xy 129.54 92.71) (xy 125.73 92.71)
 		)
@@
 	(wire
 		(pts
-			(xy 187.96 71.12) (xy 193.04 71.12)
-		)
-		(stroke
-			(width 0)
-			(type default)
-		)
-	)
-	(wire
-		(pts
-			(xy 193.04 78.74) (xy 193.04 81.28)
+			(xy 187.96 71.12) (xy 195.58 71.12)
 		)
 		(stroke
@@
 	(wire
 		(pts
-			(xy 187.96 78.74) (xy 193.04 78.74)
-		)
-		(stroke
-			(width 0)
-			(type default)
-		)
-	)
-	(wire
-		(pts
 			(xy 181.61 71.12) (xy 187.96 71.12)
 		)
@@
 		(pts
 			(xy 181.61 91.44) (xy 181.61 95.25)
+		)
+		(stroke
+			(width 0)
+			(type default)
+		)
+	)
+	(wire
+		(pts
+			(xy 187.96 78.74) (xy 187.96 81.28)
 		)
 		(stroke
@@
 	(symbol
 		(lib_id "power:GND")
-		(at 193.04 81.28 0)
+		(at 187.96 81.28 0)
 		(unit 1)
 		(exclude_from_sim no)
@@
 		(fields_autoplaced yes)
 		(property "Reference" "#PWR086"
-			(at 193.04 87.63 0)
+			(at 187.96 87.63 0)
 			(effects
 				(font
@@
 		)
 		(property "Value" "GND"
-			(at 193.04 86.36 0)
-			(effects
-				(font
-					(size 1.27 1.27)
-				)
-			)
-		)
-		(property "Footprint" ""
-			(at 193.04 81.28 0)
+			(at 187.96 86.36 0)
+			(effects
+				(font
+					(size 1.27 1.27)
+				)
+			)
+		)
+		(property "Footprint" ""
+			(at 187.96 81.28 0)
 			(effects
 				(font
@@
 		)
 		(property "Datasheet" ""
-			(at 193.04 81.28 0)
+			(at 187.96 81.28 0)
 			(effects
 				(font
@@
 		)
 		(property "Description" "Power symbol creates a global label with name \"GND\" , ground"
-			(at 193.04 81.28 0)
+			(at 187.96 81.28 0)
 			(effects
 				(font
@@
 					(unit 1)
 				)
-			)
-		)
-	)
-	(symbol
-		(lib_id "Device:Battery_Cell")
-		(at 193.04 76.2 0)
-		(unit 1)
-		(exclude_from_sim no)
-		(in_bom yes)
-		(on_board yes)
-		(dnp no)
-		(fields_autoplaced yes)
-		(property "Reference" "BT2"
-			(at 196.85 73.0884 0)
-			(effects
-				(font
-					(size 1.27 1.27)
-				)
-				(justify left)
-			)
-		)
-		(property "Value" "Battery_Cell"
-			(at 196.85 75.6284 0)
-			(effects
-				(font
-					(size 1.27 1.27)
-				)
-				(justify left)
-			)
-		)
-		(property "Footprint" ""
-			(at 193.04 74.676 90)
-			(effects
-				(font
-					(size 1.27 1.27)
-				)
-				(hide yes)
-			)
-		)
-		(property "Datasheet" "~"
-			(at 193.04 74.676 90)
-			(effects
-				(font
-					(size 1.27 1.27)
-				)
-				(hide yes)
-			)
-		)
-		(property "Description" "Single-cell battery"
-			(at 193.04 76.2 0)
-			(effects
-				(font
-					(size 1.27 1.27)
-				)
-				(hide yes)
-			)
-		)
-		(pin "1"
-		)
-		(pin "2"
-		)
-		(instances
-			(project ""
-				(path "/52181fb0-1be8-41da-83b2-7d5a62778ff4/b9fa46c4-d87c-4f12-b237-f801e8270b19"
-					(reference "BT2")
-					(unit 1)
-				)

Commit message: Minor Changes
Parts:
- removed R31: R, symbol Device:R
- C23: renamed from C25; value C -> 2025Fp
- C25: renamed from C23; value CBAT -> 1UF
- renumbered R33 to R30, R32 to R31, R34 to R32, U21 to U23, U19 to U24
Changed lines of the file:
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@@
-	)
-	(junction
-		(at 181.61 71.12)
-		(diameter 0)
-		(color 0 0 0 0)
 	)
 	(junction
@@
 	(wire
 		(pts
-			(xy 181.61 71.12) (xy 181.61 83.82)
-		)
-		(stroke
-			(width 0)
-			(type default)
-		)
-	)
-	(wire
-		(pts
 			(xy 129.54 92.71) (xy 125.73 92.71)
 		)
@@
 	(wire
 		(pts
-			(xy 177.8 71.12) (xy 181.61 71.12)
+			(xy 177.8 71.12) (xy 187.96 71.12)
 		)
 		(stroke
@@
 	(wire
 		(pts
-			(xy 181.61 71.12) (xy 187.96 71.12)
-		)
-		(stroke
-			(width 0)
-			(type default)
-		)
-	)
-	(wire
-		(pts
 			(xy 115.57 99.06) (xy 120.65 99.06)
 		)
@@
 		(pts
 			(xy 111.76 101.6) (xy 129.54 101.6)
-		)
-		(stroke
-			(width 0)
-			(type default)
-		)
-	)
-	(wire
-		(pts
-			(xy 181.61 91.44) (xy 181.61 95.25)
-		)
-		(stroke
-			(width 0)
-			(type default)
-		)
-	)
-	(wire
-		(pts
-			(xy 187.96 78.74) (xy 187.96 81.28)
 		)
 		(stroke
@@
 		(dnp no)
 		(fields_autoplaced yes)
-		(property "Reference" "#PWR092"
+		(property "Reference" "#PWR091"
 			(at 125.73 90.17 0)
 			(effects
@@
 			(project ""
 				(path "/52181fb0-1be8-41da-83b2-7d5a62778ff4/b9fa46c4-d87c-4f12-b237-f801e8270b19"
-					(reference "#PWR092")
+					(reference "#PWR091")
 					(unit 1)
 				)
@@
 		(dnp no)
 		(fields_autoplaced yes)
-		(property "Reference" "#PWR088"
+		(property "Reference" "#PWR094"
 			(at 176.53 110.49 0)
 			(effects
@@
 			(project "Smarter Watch Stuff"
 				(path "/52181fb0-1be8-41da-83b2-7d5a62778ff4/b9fa46c4-d87c-4f12-b237-f801e8270b19"
-					(reference "#PWR088")
+					(reference "#PWR094")
 					(unit 1)
 				)
@@
 	)
 	(symbol
-		(lib_id "Device:R")
-		(at 181.61 87.63 0)
-		(unit 1)
-		(exclude_from_sim no)
-		(in_bom yes)
-		(on_board yes)
-		(dnp no)
-		(fields_autoplaced yes)
-		(property "Reference" "R31"
-			(at 184.15 86.3599 0)
-			(effects
-				(font
-					(size 1.27 1.27)
-				)
-				(justify left)
-			)
-		)
-		(property "Value" "R"
-			(at 184.15 88.8999 0)
-			(effects
-				(font
-					(size 1.27 1.27)
-				)
-				(justify left)
-			)
-		)
-		(property "Footprint" ""
-			(at 179.832 87.63 90)
-			(effects
-				(font
-					(size 1.27 1.27)
-				)
-				(hide yes)
-			)
-		)
-		(property "Datasheet" "~"
-			(at 181.61 87.63 0)
-			(effects
-				(font
-					(size 1.27 1.27)
-				)
-				(hide yes)
-			)
-		)
-		(property "Description" "Resistor"
-			(at 181.61 87.63 0)
-			(effects
-				(font
-					(size 1.27 1.27)
-				)
-				(hide yes)
-			)
-		)
-		(pin "2"
-		)
-		(pin "1"
-		)
-		(instances
-			(project ""
-				(path "/52181fb0-1be8-41da-83b2-7d5a62778ff4/b9fa46c4-d87c-4f12-b237-f801e8270b19"
-					(reference "R31")
-					(unit 1)
-				)
-			)
-		)
-	)
-	(symbol
 		(lib_id "Custom:OpenJumper")
 		(at 93.98 100.33 180)
@@
 		(dnp no)
 		(fields_autoplaced yes)
-		(property "Reference" "U21"
+		(property "Reference" "U23"
 			(at 93.98 102.87 0)
 			(effects
@@
 			(project "Smarter Watch Stuff"
 				(path "/52181fb0-1be8-41da-83b2-7d5a62778ff4/b9fa46c4-d87c-4f12-b237-f801e8270b19"
-					(reference "U21")
+					(reference "U23")
 					(unit 1)
 				)
@@
 		(dnp no)
 		(fields_autoplaced yes)
-		(property "Reference" "#PWR084"
+		(property "Reference" "#PWR092"
 			(at 123.19 90.17 0)
 			(effects
@@
 			(project ""
 				(path "/52181fb0-1be8-41da-83b2-7d5a62778ff4/b9fa46c4-d87c-4f12-b237-f801e8270b19"
-					(reference "#PWR084")
+					(reference "#PWR092")
 					(unit 1)
 				)
@@
 		(dnp no)
 		(fields_autoplaced yes)
-		(property "Reference" "#PWR094"
+		(property "Reference" "#PWR090"
 			(at 109.22 71.12 0)
 			(effects
@@
 			(project "Smarter Watch Stuff"
 				(path "/52181fb0-1be8-41da-83b2-7d5a62778ff4/b9fa46c4-d87c-4f12-b237-f801e8270b19"
-					(reference "#PWR094")
+					(reference "#PWR090")
 					(unit 1)
 				)
@@
 	(symbol
 		(lib_id "power:GND")
-		(at 187.96 81.28 0)
-		(unit 1)
-		(exclude_from_sim no)
-		(in_bom yes)
-		(on_board yes)
-		(dnp no)
-		(fields_autoplaced yes)
-		(property "Reference" "#PWR086"
-			(at 187.96 87.63 0)
+		(at 187.96 78.74 0)
+		(unit 1)
+		(exclude_from_sim no)
+		(in_bom yes)
+		(on_board yes)
+		(dnp no)
+		(fields_autoplaced yes)
+		(property "Reference" "#PWR096"
+			(at 187.96 85.09 0)
 			(effects
 				(font
@@
 		)
 		(property "Value" "GND"
-			(at 187.96 86.36 0)
-			(effects
-				(font
-					(size 1.27 1.27)
-				)
-			)
-		)
-		(property "Footprint" ""
-			(at 187.96 81.28 0)
+			(at 187.96 83.82 0)
+			(effects
+				(font
+					(size 1.27 1.27)
+				)
+			)
+		)
+		(property "Footprint" ""
+			(at 187.96 78.74 0)
 			(effects
 				(font
@@
 		)
 		(property "Datasheet" ""
-			(at 187.96 81.28 0)
+			(at 187.96 78.74 0)
 			(effects
 				(font
@@
 		)
 		(property "Description" "Power symbol creates a global label with name \"GND\" , ground"
-			(at 187.96 81.28 0)
+			(at 187.96 78.74 0)
 			(effects
 				(font
@@
 			(project ""
 				(path "/52181fb0-1be8-41da-83b2-7d5a62778ff4/b9fa46c4-d87c-4f12-b237-f801e8270b19"
-					(reference "#PWR086")
+					(reference "#PWR096")
 					(unit 1)
 				)
@@
 		(dnp no)
 		(fields_autoplaced yes)
-		(property "Reference" "C25"
+		(property "Reference" "C23"
 			(at 119.38 63.5 90)
 			(effects
@@
 			)
 		)
-		(property "Value" "C"
+		(property "Value" "2025Fp"
 			(at 119.38 66.04 90)
 			(effects
@@
 			(project ""
 				(path "/52181fb0-1be8-41da-83b2-7d5a62778ff4/b9fa46c4-d87c-4f12-b237-f801e8270b19"
-					(reference "C25")
+					(reference "C23")
 					(unit 1)
 				)
@@
 		(dnp no)
 		(fields_autoplaced yes)
-		(property "Reference" "#PWR087"
+		(property "Reference" "#PWR097"
 			(at 194.31 100.33 0)
 			(effects
@@
 			(project "Smarter Watch Stuff"
 				(path "/52181fb0-1be8-41da-83b2-7d5a62778ff4/b9fa46c4-d87c-4f12-b237-f801e8270b19"
-					(reference "#PWR087")
+					(reference "#PWR097")
 					(unit 1)
 				)
@@
 		(dnp no)
 		(fields_autoplaced yes)
-		(property "Reference" "C23"
+		(property "Reference" "C25"
 			(at 191.77 73.6599 0)
 			(effects
@@
 			)
 		)
-		(property "Value" "CBAT"
+		(property "Value" "1UF"
 			(at 191.77 76.1999 0)
 			(effects
@@
 			(project ""
 				(path "/52181fb0-1be8-41da-83b2-7d5a62778ff4/b9fa46c4-d87c-4f12-b237-f801e8270b19"
-					(reference "C23")
+					(reference "C25")
 					(unit 1)
 				)
@@
 		(dnp no)
 		(fields_autoplaced yes)
-		(property "Reference" "U19"
+		(property "Reference" "U24"
 			(at 149.86 67.31 0)
 			(effects
@@
 			(project ""
 				(path "/52181fb0-1be8-41da-83b2-7d5a62778ff4/b9fa46c4-d87c-4f12-b237-f801e8270b19"
-					(reference "U19")
+					(reference "U24")
 					(unit 1)
 				)
@@
 		(dnp no)
 		(fields_autoplaced yes)
-		(property "Reference" "#PWR090"
+		(property "Reference" "#PWR093"
 			(at 176.53 107.95 0)
 			(effects
@@
 			(project "Smarter Watch Stuff"
 				(path "/52181fb0-1be8-41da-83b2-7d5a62778ff4/b9fa46c4-d87c-4f12-b237-f801e8270b19"
-					(reference "#PWR090")
+					(reference "#PWR093")
 					(unit 1)
 				)
@@
 		(dnp no)
 		(fields_autoplaced yes)
-		(property "Reference" "#PWR093"
+		(property "Reference" "#PWR088"
 			(at 92.71 97.79 0)
 			(effects
@@
 			(project "Smarter Watch Stuff"
 				(path "/52181fb0-1be8-41da-83b2-7d5a62778ff4/b9fa46c4-d87c-4f12-b237-f801e8270b19"
-					(reference "#PWR093")
+					(reference "#PWR088")
 					(unit 1)
 				)
@@
 		(dnp no)
 		(fields_autoplaced yes)
-		(property "Reference" "#PWR085"
+		(property "Reference" "#PWR098"
 			(at 191.77 71.12 0)
 			(effects
@@
 			(project ""
 				(path "/52181fb0-1be8-41da-83b2-7d5a62778ff4/b9fa46c4-d87c-4f12-b237-f801e8270b19"
-					(reference "#PWR085")
+					(reference "#PWR098")
 					(unit 1)
 				)
@@
 		(dnp no)
 		(fields_autoplaced yes)
-		(property "Reference" "#PWR091"
+		(property "Reference" "#PWR089"
 			(at 111.76 82.55 0)
 			(effects
@@
 			(project "Smarter Watch Stuff"
 				(path "/52181fb0-1be8-41da-83b2-7d5a62778ff4/b9fa46c4-d87c-4f12-b237-f801e8270b19"
-					(reference "#PWR091")
+					(reference "#PWR089")
 					(unit 1)
 				)
@@
 		(dnp no)
 		(fields_autoplaced yes)
-		(property "Reference" "R32"
+		(property "Reference" "R31"
 			(at 113.03 96.5201 0)
 			(effects
@@
 			(project "Smarter Watch Stuff"
 				(path "/52181fb0-1be8-41da-83b2-7d5a62778ff4/b9fa46c4-d87c-4f12-b237-f801e8270b19"
-					(reference "R32")
+					(reference "R31")
 					(unit 1)
 				)
@@
 		(dnp no)
 		(fields_autoplaced yes)
-		(property "Reference" "R33"
+		(property "Reference" "R30"
 			(at 109.22 99.0601 0)
 			(effects
@@
 			(project "Smarter Watch Stuff"
 				(path "/52181fb0-1be8-41da-83b2-7d5a62778ff4/b9fa46c4-d87c-4f12-b237-f801e8270b19"
-					(reference "R33")
+					(reference "R30")
 					(unit 1)
 				)
@@
 		(dnp no)
 		(fields_autoplaced yes)
-		(property "Reference" "R34"
+		(property "Reference" "R32"
 			(at 119.38 74.93 90)
 			(effects
@@
 			(project ""
 				(path "/52181fb0-1be8-41da-83b2-7d5a62778ff4/b9fa46c4-d87c-4f12-b237-f801e8270b19"
-					(reference "R34")
+					(reference "R32")
 					(unit 1)
 				)
@@
 		(dnp no)
 		(fields_autoplaced yes)
-		(property "Reference" "#PWR089"
+		(property "Reference" "#PWR095"
 			(at 179.07 88.9 0)
 			(effects
@@
 			(project "Smarter Watch Stuff"
 				(path "/52181fb0-1be8-41da-83b2-7d5a62778ff4/b9fa46c4-d87c-4f12-b237-f801e8270b19"
-					(reference "#PWR089")
-					(unit 1)
-				)
+					(reference "#PWR095")
+					(unit 1)
+				)

Commit message: foot print stuff
Parts:
- C23, C24, C25: footprint (none) -> Capacitor_SMD:C_0402_1005Metric
- R30, R31: footprint (none) -> Resistor_SMD:R_0402_1005Metric
- R32: value R -> 10k; footprint (none) -> Resistor_SMD:R_0402_1005Metric
Changed lines of the file:
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@@
 			)
 		)
-		(property "Footprint" ""
+		(property "Footprint" "Capacitor_SMD:C_0402_1005Metric"
 			(at 187.96 99.3648 0)
 			(effects
@@
 			)
 		)
-		(property "Footprint" ""
+		(property "Footprint" "Capacitor_SMD:C_0402_1005Metric"
 			(at 123.19 70.1548 0)
 			(effects
@@
 			)
 		)
-		(property "Footprint" ""
+		(property "Footprint" "Capacitor_SMD:C_0402_1005Metric"
 			(at 188.9252 78.74 0)
 			(effects
@@
 			)
 		)
-		(property "Footprint" ""
+		(property "Footprint" "Resistor_SMD:R_0402_1005Metric"
 			(at 117.348 95.25 90)
 			(effects
@@
 			)
 		)
-		(property "Footprint" ""
+		(property "Footprint" "Resistor_SMD:R_0402_1005Metric"
 			(at 113.538 97.79 90)
 			(effects
@@
 			)
 		)
-		(property "Value" "R"
+		(property "Value" "10k"
 			(at 119.38 77.47 90)
 			(effects
@@
 			)
 		)
-		(property "Footprint" ""
+		(property "Footprint" "Resistor_SMD:R_0402_1005Metric"
 			(at 119.38 83.058 90)
 			(effects

Commit message: Footprint Stuff
Parts:
- U24: footprint AS3935-BQFT:QFN65P400X400X80-17N -> (none)
Changed lines of the file:
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@@
 			)
 		)
-		(property "Footprint" "AS3935-BQFT:QFN65P400X400X80-17N"
+		(property "Footprint" ""
 			(at 149.86 92.71 0)
 			(effects

Commit message: Jumpers
Parts:
- U22, U23: footprint (none) -> Custom_Foot:Jumper_NO
Changed lines of the file:
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@@
 			)
 		)
-		(property "Footprint" ""
+		(property "Footprint" "Custom_Foot:Jumper_NO"
 			(at 93.98 100.33 0)
 			(effects
@@
 			)
 		)
-		(property "Footprint" ""
+		(property "Footprint" "Custom_Foot:Jumper_NO"
 			(at 93.98 92.71 0)
 			(effects

Commit message: footprint
Parts:
- U24: footprint (none) -> Custom_Foot:QFN65P400X400X80-17N
Changed lines of the file:
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@@
 			)
 		)
-		(property "Footprint" ""
+		(property "Footprint" "Custom_Foot:QFN65P400X400X80-17N"
 			(at 149.86 92.71 0)
 			(effects
