File: SmarterWatch_KiCad/Lightning.kicad_sch (KiCad schematic)
At the start: 10 parts, among them U24 AS3935-BQFT

Commit message: New custom foot and assignments
Parts:
- L1: footprint (none) -> Custom_Foot:Antenna_MA5532-AE
Changed lines of the file:
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@@
 			)
 		)
-		(property "Footprint" ""
+		(property "Footprint" "Custom_Foot:Antenna_MA5532-AE"
 			(at 119.38 67.31 0)
 			(effects

Commit message: FINAL
Parts:
- U22, U23: value ~ -> (none)
