File: SmarterWatch_KiCad/Skin.kicad_sch (KiCad schematic)
At the start: 9 parts, among them U14 MAX30205MTA+T

Commit message: order
Parts:
- C20: footprint (none) -> Capacitor_SMD:C_01005_0402Metric
Changed lines of the file:
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@@
 			)
 		)
-		(property "Footprint" ""
+		(property "Footprint" "Capacitor_SMD:C_01005_0402Metric"
 			(at 160.02 95.5548 0)
 			(effects

Commit message: Minor Changes
Parts:
- renumbered R29 to R26, R28 to R27, R27 to R28, R26 to R29, U14 to U17, U16 to U18, U15 to U19, U17 to U20
Changed lines of the file:
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@@
 		(dnp no)
 		(fields_autoplaced yes)
-		(property "Reference" "U16"
+		(property "Reference" "U18"
 			(at 167.64 92.71 0)
 			(effects
@@
 			(project "Smarter Watch Stuff"
 				(path "/52181fb0-1be8-41da-83b2-7d5a62778ff4/596be1bd-3875-49a3-8dbd-4c169cd37f92"
-					(reference "U16")
+					(reference "U18")
 					(unit 1)
 				)
@@
 		(dnp no)
 		(fields_autoplaced yes)
-		(property "Reference" "U14"
+		(property "Reference" "U17"
 			(at 119.38 83.82 0)
 			(effects
@@
 			(project ""
 				(path "/52181fb0-1be8-41da-83b2-7d5a62778ff4/596be1bd-3875-49a3-8dbd-4c169cd37f92"
-					(reference "U14")
+					(reference "U17")
 					(unit 1)
 				)
@@
 		(dnp no)
 		(fields_autoplaced yes)
-		(property "Reference" "#PWR070"
+		(property "Reference" "#PWR078"
 			(at 149.86 120.65 0)
 			(effects
@@
 			(project ""
 				(path "/52181fb0-1be8-41da-83b2-7d5a62778ff4/596be1bd-3875-49a3-8dbd-4c169cd37f92"
-					(reference "#PWR070")
+					(reference "#PWR078")
 					(unit 1)
 				)
@@
 		(dnp no)
 		(fields_autoplaced yes)
-		(property "Reference" "#PWR072"
+		(property "Reference" "#PWR077"
 			(at 153.67 93.98 0)
 			(effects
@@
 			(project ""
 				(path "/52181fb0-1be8-41da-83b2-7d5a62778ff4/596be1bd-3875-49a3-8dbd-4c169cd37f92"
-					(reference "#PWR072")
+					(reference "#PWR077")
 					(unit 1)
 				)
@@
 		(dnp no)
 		(fields_autoplaced yes)
-		(property "Reference" "R28"
+		(property "Reference" "R27"
 			(at 148.59 106.6799 0)
 			(effects
@@
 			(project "Smarter Watch Stuff"
 				(path "/52181fb0-1be8-41da-83b2-7d5a62778ff4/596be1bd-3875-49a3-8dbd-4c169cd37f92"
-					(reference "R28")
+					(reference "R27")
 					(unit 1)
 				)
@@
 		(dnp no)
 		(fields_autoplaced yes)
-		(property "Reference" "#PWR073"
+		(property "Reference" "#PWR080"
 			(at 168.91 105.41 0)
 			(effects
@@
 			(project ""
 				(path "/52181fb0-1be8-41da-83b2-7d5a62778ff4/596be1bd-3875-49a3-8dbd-4c169cd37f92"
-					(reference "#PWR073")
+					(reference "#PWR080")
 					(unit 1)
 				)
@@
 		(dnp no)
 		(fields_autoplaced yes)
-		(property "Reference" "#PWR075"
+		(property "Reference" "#PWR076"
 			(at 143.51 88.9 0)
 			(effects
@@
 			(project ""
 				(path "/52181fb0-1be8-41da-83b2-7d5a62778ff4/596be1bd-3875-49a3-8dbd-4c169cd37f92"
-					(reference "#PWR075")
+					(reference "#PWR076")
 					(unit 1)
 				)
@@
 		(dnp no)
 		(fields_autoplaced yes)
-		(property "Reference" "R26"
+		(property "Reference" "R29"
 			(at 157.48 101.5999 0)
 			(effects
@@
 			(project ""
 				(path "/52181fb0-1be8-41da-83b2-7d5a62778ff4/596be1bd-3875-49a3-8dbd-4c169cd37f92"
-					(reference "R26")
+					(reference "R29")
 					(unit 1)
 				)
@@
 		(dnp no)
 		(fields_autoplaced yes)
-		(property "Reference" "#PWR071"
+		(property "Reference" "#PWR075"
 			(at 90.17 116.84 0)
 			(effects
@@
 			(project ""
 				(path "/52181fb0-1be8-41da-83b2-7d5a62778ff4/596be1bd-3875-49a3-8dbd-4c169cd37f92"
-					(reference "#PWR071")
+					(reference "#PWR075")
 					(unit 1)
 				)
@@
 		(dnp no)
 		(fields_autoplaced yes)
-		(property "Reference" "R27"
+		(property "Reference" "R28"
 			(at 152.4 104.1399 0)
 			(effects
@@
 			(project "Smarter Watch Stuff"
 				(path "/52181fb0-1be8-41da-83b2-7d5a62778ff4/596be1bd-3875-49a3-8dbd-4c169cd37f92"
-					(reference "R27")
+					(reference "R28")
 					(unit 1)
 				)
@@
 		(dnp no)
 		(fields_autoplaced yes)
-		(property "Reference" "U15"
+		(property "Reference" "U19"
 			(at 167.64 100.33 0)
 			(effects
@@
 			(project "Smarter Watch Stuff"
 				(path "/52181fb0-1be8-41da-83b2-7d5a62778ff4/596be1bd-3875-49a3-8dbd-4c169cd37f92"
-					(reference "U15")
+					(reference "U19")
 					(unit 1)
 				)
@@
 		(dnp no)
 		(fields_autoplaced yes)
-		(property "Reference" "#PWR074"
+		(property "Reference" "#PWR079"
 			(at 166.37 96.52 0)
 			(effects
@@
 			(project "Smarter Watch Stuff"
 				(path "/52181fb0-1be8-41da-83b2-7d5a62778ff4/596be1bd-3875-49a3-8dbd-4c169cd37f92"
-					(reference "#PWR074")
+					(reference "#PWR079")
 					(unit 1)
 				)
@@
 		(dnp no)
 		(fields_autoplaced yes)
-		(property "Reference" "#PWR076"
+		(property "Reference" "#PWR074"
 			(at 83.82 99.06 0)
 			(effects
@@
 			(project "Smarter Watch Stuff"
 				(path "/52181fb0-1be8-41da-83b2-7d5a62778ff4/596be1bd-3875-49a3-8dbd-4c169cd37f92"
-					(reference "#PWR076")
+					(reference "#PWR074")
 					(unit 1)
 				)
@@
 		(dnp no)
 		(fields_autoplaced yes)
-		(property "Reference" "R29"
+		(property "Reference" "R26"
 			(at 83.82 92.71 90)
 			(effects
@@
 			(project ""
 				(path "/52181fb0-1be8-41da-83b2-7d5a62778ff4/596be1bd-3875-49a3-8dbd-4c169cd37f92"
-					(reference "R29")
+					(reference "R26")
 					(unit 1)
 				)
@@
 		(dnp no)
 		(fields_autoplaced yes)
-		(property "Reference" "U17"
+		(property "Reference" "U20"
 			(at 167.64 107.95 0)
 			(effects
@@
 			(project "Smarter Watch Stuff"
 				(path "/52181fb0-1be8-41da-83b2-7d5a62778ff4/596be1bd-3875-49a3-8dbd-4c169cd37f92"
-					(reference "U17")
-					(unit 1)
-				)
+					(reference "U20")
+					(unit 1)
+				)

Commit message: foot print stuff
Parts:
- R26, R27, R28, R29: footprint (none) -> Resistor_SMD:R_0402_1005Metric
Changed lines of the file:
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@@
 			)
 		)
-		(property "Footprint" ""
+		(property "Footprint" "Resistor_SMD:R_0402_1005Metric"
 			(at 144.272 107.95 90)
 			(effects
@@
 			)
 		)
-		(property "Footprint" ""
+		(property "Footprint" "Resistor_SMD:R_0402_1005Metric"
 			(at 156.718 102.87 90)
 			(effects
@@
 			)
 		)
-		(property "Footprint" ""
+		(property "Footprint" "Resistor_SMD:R_0402_1005Metric"
 			(at 148.082 105.41 90)
 			(effects
@@
 			)
 		)
-		(property "Footprint" ""
+		(property "Footprint" "Resistor_SMD:R_0402_1005Metric"
 			(at 83.82 100.838 90)
 			(effects

Commit message: Footprint Stuff
Parts:
- U17: footprint 21-0137_T833+2_MXM -> (none)
Changed lines of the file:
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@@
 			)
 		)
-		(property "Footprint" "21-0137_T833+2_MXM"
+		(property "Footprint" ""
 			(at 99.06 93.98 0)
 			(effects

Commit message: Foot
Parts:
- U17: footprint (none) -> Custom_Foot:XDCR_MAX30101EFD_
Changed lines of the file:
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@@
 			)
 		)
-		(property "Footprint" ""
+		(property "Footprint" "Custom_Foot:XDCR_MAX30101EFD_"
 			(at 99.06 93.98 0)
 			(effects

Commit message: Jumpers
Parts:
- U18, U19, U20: footprint (none) -> Custom_Foot:Jumper_NO
Changed lines of the file:
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@@
 			)
 		)
-		(property "Footprint" ""
+		(property "Footprint" "Custom_Foot:Jumper_NO"
 			(at 167.64 95.25 0)
 			(effects
@@
 			)
 		)
-		(property "Footprint" ""
+		(property "Footprint" "Custom_Foot:Jumper_NO"
 			(at 167.64 102.87 0)
 			(effects
@@
 			)
 		)
-		(property "Footprint" ""
+		(property "Footprint" "Custom_Foot:Jumper_NO"
 			(at 167.64 110.49 0)
 			(effects

Commit message: Label Jumpers
Parts:
- U17: footprint Custom_Foot:XDCR_MAX30101EFD_ -> (none)
- U18, U19, U20: footprint Custom_Foot:Jumper_NO -> (none)
Changed lines of the file:
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@@
 			)
 		)
-		(property "Footprint" "Custom_Foot:Jumper_NO"
+		(property "Footprint" ""
 			(at 167.64 95.25 0)
 			(effects
@@
 			)
 		)
-		(property "Footprint" "Custom_Foot:XDCR_MAX30101EFD_"
+		(property "Footprint" ""
 			(at 99.06 93.98 0)
 			(effects
@@
 			)
 		)
-		(property "Footprint" "Custom_Foot:Jumper_NO"
+		(property "Footprint" ""
 			(at 167.64 102.87 0)
 			(effects
@@
 			)
 		)
-		(property "Footprint" "Custom_Foot:Jumper_NO"
+		(property "Footprint" ""
 			(at 167.64 110.49 0)
 			(effects

Commit message: added pad to symbol
Parts:
- U17: footprint (none) -> Custom_Foot:XDCR_MAX30101EFD_
- U18, U19, U20: footprint (none) -> Custom_Foot:Jumper_NO
Changed lines of the file:
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@@
 			)
 		)
-		(property "Footprint" ""
+		(property "Footprint" "Custom_Foot:Jumper_NO"
 			(at 167.64 95.25 0)
 			(effects
@@
 			)
 		)
-		(property "Footprint" ""
+		(property "Footprint" "Custom_Foot:XDCR_MAX30101EFD_"
 			(at 99.06 93.98 0)
 			(effects
@@
 			)
 		)
-		(property "Footprint" ""
+		(property "Footprint" "Custom_Foot:Jumper_NO"
 			(at 167.64 102.87 0)
 			(effects
@@
 			)
 		)
-		(property "Footprint" ""
+		(property "Footprint" "Custom_Foot:Jumper_NO"
 			(at 167.64 110.49 0)
 			(effects
