File: SmarterWatch_KiCad/Skin.kicad_sch (KiCad schematic)
At the start: 9 parts, among them U17 MAX30205MTA+T

Commit message: update
Parts:
- U17: footprint Custom_Foot:XDCR_MAX30101EFD_ -> Custom_Foot:SON65P300X300X80-9N
Changed lines of the file:
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@@
 			)
 		)
-		(property "Footprint" "Custom_Foot:XDCR_MAX30101EFD_"
+		(property "Footprint" "Custom_Foot:SON65P300X300X80-9N"
 			(at 99.06 93.98 0)
 			(effects

Commit message: FINAL
Parts:
- U18, U19, U20: value ~ -> (none)
