File: SmarterWatch_KiCad/Spo2.kicad_sch (KiCad schematic)
At the start: 7 parts, among them U10 MAX30102, U9 MIC5365-1.8YC5

Commit message: via stuff
Connections:
- net +3.3V_sensor renamed +3.3V
Changed lines of the file:
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@@
 		)
 	)
-	(global_label "+3.3V_sensor"
-		(shape input)
-		(at 134.62 76.2 90)
+	(symbol
+		(lib_id "power:+3.3V")
+		(at 134.62 76.2 0)
+		(unit 1)
+		(exclude_from_sim no)
+		(in_bom yes)
+		(on_board yes)
+		(dnp no)
 		(fields_autoplaced yes)
-		(effects
-			(font
-				(size 1.27 1.27)
-			)
-			(justify left)
-		)
-		(property "Intersheetrefs" "${INTERSHEET_REFS}"
-			(at 134.62 60.3334 90)
+		(property "Reference" "#PWR0108"
+			(at 134.62 80.01 0)
 			(effects
 				(font
 					(size 1.27 1.27)
 				)
-				(justify left)
 				(hide yes)
 			)
 		)
+		(property "Value" "+3.3V"
+			(at 134.62 71.12 0)
+			(effects
+				(font
+					(size 1.27 1.27)
+				)
+			)
+		)
+		(property "Footprint" ""
+			(at 134.62 76.2 0)
+			(effects
+				(font
+					(size 1.27 1.27)
+				)
+				(hide yes)
+			)
+		)
+		(property "Datasheet" ""
+			(at 134.62 76.2 0)
+			(effects
+				(font
+					(size 1.27 1.27)
+				)
+				(hide yes)
+			)
+		)
+		(property "Description" "Power symbol creates a global label with name \"+3.3V\""
+			(at 134.62 76.2 0)
+			(effects
+				(font
+					(size 1.27 1.27)
+				)
+				(hide yes)
+			)
+		)
+		(pin "1"
+		)
+		(instances
+			(project ""
+				(path "/52181fb0-1be8-41da-83b2-7d5a62778ff4/ede32b43-0075-4e9b-9527-55f10148fcb6"
+					(reference "#PWR0108")
+					(unit 1)
+				)
+			)
+		)
