File: SmarterWatch_KiCad/RGB.kicad_sch (KiCad schematic)
At the start: 1 part

Commit message: sync
Parts:
- D2: footprint Custom_Foot:LED_IN-PI554FCH -> (none)
Changed lines of the file:
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@@
 			)
 		)
-		(property "Footprint" "Custom_Foot:LED_IN-PI554FCH"
+		(property "Footprint" ""
 			(at 144.78 106.68 0)
 			(effects
