File: SmarterWatch_KiCad/RGB.kicad_sch (KiCad schematic)
At the start: 1 part

Commit message: Footprint Stuff
Parts:
- D2: footprint LED_SMD:LED_Inolux_IN-PI554FCH_PLCC4_5.0x5.0mm_P3.2mm -> (none)
Changed lines of the file:
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@@
 			)
 		)
-		(property "Footprint" "LED_SMD:LED_Inolux_IN-PI554FCH_PLCC4_5.0x5.0mm_P3.2mm"
+		(property "Footprint" ""
 			(at 144.78 106.68 0)
 			(effects

Commit message: footprints
Parts:
- D2: footprint (none) -> Custom_Foot:LED_IN-PI554FCH
Changed lines of the file:
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@@
 			)
 		)
-		(property "Footprint" ""
+		(property "Footprint" "Custom_Foot:LED_IN-PI554FCH"
 			(at 144.78 106.68 0)
 			(effects
