File: SmarterWatch_KiCad/Level_Shifter.kicad_sch (KiCad schematic)
At the start: 4 parts

Commit message: Minor Changes
Parts:
- renumbered R37 to R36, R38 to R37, U23 to U26
Changed lines of the file:
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@@
 		(dnp no)
 		(fields_autoplaced yes)
-		(property "Reference" "R38"
+		(property "Reference" "R37"
 			(at 151.13 86.3599 0)
 			(effects
@@
 			(project "Smarter Watch Stuff"
 				(path "/52181fb0-1be8-41da-83b2-7d5a62778ff4/a7d1cf48-cec0-4485-89d4-6b86e8a98aaa"
-					(reference "R38")
+					(reference "R37")
 					(unit 1)
 				)
@@
 		(dnp no)
 		(fields_autoplaced yes)
-		(property "Reference" "#PWR0104"
+		(property "Reference" "#PWR0105"
 			(at 148.59 87.63 0)
 			(effects
@@
 			(project "Smarter Watch Stuff"
 				(path "/52181fb0-1be8-41da-83b2-7d5a62778ff4/a7d1cf48-cec0-4485-89d4-6b86e8a98aaa"
-					(reference "#PWR0104")
+					(reference "#PWR0105")
 					(unit 1)
 				)
@@
 		(dnp no)
 		(fields_autoplaced yes)
-		(property "Reference" "#PWR0105"
+		(property "Reference" "#PWR0104"
 			(at 130.81 119.38 0)
 			(effects
@@
 			(project ""
 				(path "/52181fb0-1be8-41da-83b2-7d5a62778ff4/a7d1cf48-cec0-4485-89d4-6b86e8a98aaa"
-					(reference "#PWR0105")
+					(reference "#PWR0104")
 					(unit 1)
 				)
@@
 		(on_board yes)
 		(dnp no)
-		(property "Reference" "R37"
+		(property "Reference" "R36"
 			(at 110.998 93.218 90)
 			(effects
@@
 			(project "Smarter Watch Stuff"
 				(path "/52181fb0-1be8-41da-83b2-7d5a62778ff4/a7d1cf48-cec0-4485-89d4-6b86e8a98aaa"
-					(reference "R37")
+					(reference "R36")
 					(unit 1)
 				)
@@
 		(on_board yes)
 		(dnp no)
-		(property "Reference" "#PWR0102"
+		(property "Reference" "#PWR0103"
 			(at 113.03 90.17 0)
 			(effects
@@
 			(project "Smarter Watch Stuff"
 				(path "/52181fb0-1be8-41da-83b2-7d5a62778ff4/a7d1cf48-cec0-4485-89d4-6b86e8a98aaa"
-					(reference "#PWR0102")
+					(reference "#PWR0103")
 					(unit 1)
 				)
@@
 		(dnp no)
 		(fields_autoplaced yes)
-		(property "Reference" "U23"
+		(property "Reference" "U26"
 			(at 130.81 87.63 0)
 			(effects
@@
 			(project ""
 				(path "/52181fb0-1be8-41da-83b2-7d5a62778ff4/a7d1cf48-cec0-4485-89d4-6b86e8a98aaa"
-					(reference "U23")
-					(unit 1)
-				)
+					(reference "U26")
+					(unit 1)
+				)

Commit message: Naming
Parts:
- U26: value ~ -> NLA9306MU3TAG
Changed lines of the file:
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@@
 			)
 		)
-		(property "Value" "~"
+		(property "Value" "NLA9306MU3TAG"
 			(at 130.81 90.17 0)
 			(effects

Commit message: sync
Parts:
- U26: footprint (none) -> Custom_Foot:UDFN8_(1.45x1mm)
Changed lines of the file:
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@@
 			)
 		)
-		(property "Footprint" ""
+		(property "Footprint" "Custom_Foot:UDFN8_(1.45x1mm)"
 			(at 130.81 91.44 0)
 			(effects

Commit message: button foot added on
Parts:
- U26: footprint Custom_Foot:UDFN8_(1.45x1mm) -> (none)
Changed lines of the file:
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@@
 			)
 		)
-		(property "Footprint" "Custom_Foot:UDFN8_(1.45x1mm)"
+		(property "Footprint" ""
 			(at 130.81 91.44 0)
 			(effects
