File: SmarterWatch_KiCad/Smarter Watch Stuff.kicad_pcb (KiCad board)
At the start: 4 copper layers, 39 x 39 mm, 111 parts, among them J5 CX70M-24P1, M1 Motor_DC, Q1 2N7002, Q2 2N7002, Q3 2N7002, Q4 2N7002, SW1 SW_SPST, SW2 SW_SPST, U1 MCP7940N-xSN, U10 MAX30102, U11 BMI160, U15 M24C64-WMN6TP, U16 IQS323001DNR, U17 MAX30205MTA+T, U2 TSL25911FN, U21 MMC5983MA, U24 AS3935-BQFT, U25 SGP40-D-R4, U26 NLA9306MU3TAG, U3 MCP73831-2-MC, U4 TCR2EE10, U5 ESP32-C6-MINI-1, U6 SHTC3, U7 TMP117xxDRV, U8 ST7735, U9 MIC5365-1.8YC5, Y1 Crystal

Commit message: Routing!
Parts:
- removed C1: 1 uf, Capacitor_SMD:C_0402_1005Metric
- removed C2, C3: 12 picoF, Capacitor_SMD:C_0402_1005Metric
- removed U1: MCP7940N-xSN, Package_SO:JEITA_SOIC-8_3.9x4.9mm_P1.27mm
- removed Y1: Crystal, Custom_Foot:XTAL_SC32S-7PF20PPM_EPS
- moved C21 97.7 mm to (87.1, 68.4), turned to 180 degrees
- moved C6 87.4 mm to (74.2, 50.8)
- moved C26 83.7 mm to (76.7, 72.6), turned to 180 degrees
- moved C16 83.7 mm to (101.3, 53.8), turned to 180 degrees
- moved C27 82.5 mm to (77.2, 76.6), turned to -90 degrees
- moved C17 80.6 mm to (104.5, 57.2)
- moved R34 79.8 mm to (77.2, 74.7), turned to -90 degrees
- moved C15 79.2 mm to (104.5, 54.7)
- moved R1 77.5 mm to (81.0, 52.3)
- moved C5 75.0 mm to (80.5, 62.3), turned to 180 degrees
- moved C14 1.65 mm to (81.1, 53.9), turned to -90 degrees
- moved R25 0.57 mm to (105.0, 52.9)
- moved R32 0.49 mm to (78.7, 73.3)
- moved U2 0.45 mm to (74.7, 77.5)
- moved U25 0.32 mm to (75.0, 74.7)
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Routing:
- net Net-(SW1-B): track 0.00 -> 52.4 mm, vias 0 -> 3
- net +3.3V: track 108.1 -> 148.7 mm, vias 9 -> 13
- net Screen_Reset: track 0.00 -> 39.1 mm, vias 0 -> 1
- net Screen_A0: track 0.00 -> 38.4 mm, vias 0 -> 1
- net SDA: track 15.5 -> 53.1 mm, vias 4 -> 9
- net Screen_CS: track 0.00 -> 35.2 mm, vias 0 -> 1
- net SCLK: track 0.00 -> 34.1 mm, vias 0 -> 2
- net GND: track 323.9 -> 357.3 mm, vias 12 -> 15
- net MOSI: track 11.3 -> 39.8 mm, vias 2 -> 3
- net Backlight: track 0.00 -> 25.0 mm, vias 0 -> 4
- net Vibrate: track 0.00 -> 22.3 mm, vias 0 -> 3
- net Net-(U15-A1): track 0.00 -> 21.5 mm, vias 0 -> 3
- net SCL: track 28.3 -> 49.5 mm, vias 0 -> 5
- net Sensor_enable: track 0.00 -> 18.6 mm, vias 0 -> 2
- net Screen_power: track 0.00 -> 18.2 mm, vias 0 -> 2
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
Commit message: DONE LAYOUT LETS GOOO
Routing:
- net RGB_DIN: track 0.00 -> 50.0 mm, vias 0 -> 2
- net Net-(SW2-B): track 8.06 -> 55.5 mm, vias 3 -> 5
- net GND: track 357.3 -> 403.0 mm, vias 15 -> 22
- net Net-(U17-A1): track 11.5 -> 55.3 mm, vias 1 -> 8
- net Net-(U17-A2): track 3.70 -> 44.0 mm, vias 1 -> 5
- net SDA: track 53.1 -> 90.4 mm, vias 9 -> 12
- net SCL: track 49.5 -> 76.8 mm, vias 5 -> 11
- net Net-(U17-A0): track 5.24 -> 31.3 mm, vias 1 -> 5
- net +3.3V_sensor: track 32.5 -> 55.5 mm, vias 4 -> 7
- net +3.3V: track 148.7 -> 171.3 mm, vias 13 -> 18
- net Net-(U15-A0): track 2.22 -> 23.6 mm, vias 0 -> 3
- net Net-(J5-PadB5): track 5.33 -> 14.2 mm, vias 2 -> 4
- net SCL 1.8V: track 7.78 -> 10.9 mm, vias 2 -> 3
- net +5V: track 25.0 -> 27.0 mm
- net +1V8: track 22.8 -> 21.6 mm
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- added copper zone on B.Cu, net GND
- added copper zone on F.Cu, net GND
- added copper zone on In1.Cu, net GND
- added copper zone on In2.Cu, net GND

Commit message: Even doner layout
Routing:
- net GND: vias 22 -> 23
Other:
- board text added: "Smarter"
- board text added: "Watch"

Commit message: Yay!
Routing:
- net Net-(U17-A1): vias 8 -> 7
Changed lines of the file:
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@@
-	)
-	(via
-		(at 92.936574 51.529418)
-		(size 0.25)
-		(drill 0.15)
-		(layers "F.Cu" "B.Cu")
-		(net 105)
 	)
 	(via

Commit message: via stuff
Parts:
- removed Q1: 2N7002, Package_TO_SOT_SMD:SOT-23
- removed R10: 1k, Resistor_SMD:R_0402_1005Metric
- removed R11: 10k, Resistor_SMD:R_0402_1005Metric
- added J6: ~, Connector_Wire:SolderWirePad_1x01_SMD_2x4mm, B.Cu at (98.6, 72.1)
Connections:
- C12 pad 2: +3.3V_sensor -> +3.3V
- C13 pad 1: +3.3V_sensor -> +3.3V
- C4 pad 1: +3.3V_sensor -> +3.3V
- C8 pad 2: +3.3V_sensor -> +3.3V
- U10 pad 10: +3.3V_sensor -> +3.3V
- U10 pad 9: +3.3V_sensor -> +3.3V
- U2 pad 5: +3.3V_sensor -> +3.3V
- U5 pad 25: Sensor_enable -> Net-(U5-IO19)
- U6 pad 1: +3.3V_sensor -> +3.3V
- U7 pad 5: +3.3V_sensor -> +3.3V
Routing:
- net +3.3V: track 171.3 -> 226.8 mm, vias 18 -> 25
- net +3.3V_sensor: track 55.5 -> 0.00 mm, vias 7 -> 0
- net Net-(U5-IO19): track 0.00 -> 23.9 mm, vias 0 -> 2
- net Sensor_enable: track 18.6 -> 0.00 mm, vias 2 -> 0
- net GND: track 403.0 -> 400.0 mm, vias 23 -> 24
- net Net-(Q1-G): track 2.81 -> 0.00 mm
- net SCLK: track 34.1 -> 36.0 mm
- net RGB_DIN: track 50.0 -> 51.3 mm
- net Net-(U17-A1): track 55.3 -> 55.5 mm, vias 7 -> 8

Commit message: Fixing a buncha vias (not done but I fixed a bunch of them)
Parts:
- moved R29 0.41 mm to (87.4, 71.3)
- moved R28 0.39 mm to (85.4, 71.3)
- moved C25 0.13 mm to (79.9, 70.2)
Routing:
- net SCL: track 76.8 -> 99.2 mm
- net Net-(U5-IO19): track 23.9 -> 11.3 mm, vias 2 -> 1
- net +3.3V: track 226.8 -> 238.6 mm, vias 25 -> 23
- net GND: track 400.0 -> 404.9 mm, vias 24 -> 23
- net Net-(U17-A2): track 44.0 -> 46.4 mm, vias 5 -> 4
- net SDA: track 90.4 -> 89.3 mm
- net Net-(U15-A2): track 18.1 -> 18.9 mm
- net Net-(U24-INP): track 13.0 -> 13.6 mm
- net Net-(U17-A1): track 55.5 -> 56.2 mm, vias 8 -> 7
- net Net-(U24-ADD1): track 21.7 -> 22.3 mm
- net Net-(SW1-B): track 52.7 -> 53.2 mm
