File: SmarterWatch_KiCad/CPU.kicad_sch (KiCad schematic)
At the start: 16 parts, among them SW1 SW_SPST, SW2 SW_SPST, U5 ESP32-C6-MINI-1

Commit message: update
Parts:
- added J7, J8: (no value), Connector_Wire:SolderWirePad_1x01_SMD_2x4mm, symbol SmarterWatch_symbols_j:Solder_pad
- added R11: 10k, Resistor_SMD:R_0402_1005Metric, symbol Device:R
- added SW3: SW_SPST, Custom_Foot:SMD_Button_6mm_SPST, symbol Switch:SW_SPST
- added U1: ESP32-S3-WROOM-1, RF_Module:ESP32-S3-WROOM-1, symbol RF_Module:ESP32-S3-WROOM-1
Connections:
- net +3.3V: now also R11.1, U1.2 (3V3)
- net GND: now also SW3.1 (A), U1.1 (GND), U1.40 (GND), U1.41 (GND)
- net USB_D+: now also U1.14 (USB_D+)
- net USB_D-: now also U1.13 (USB_D-)
- new net: J8.1, U1.36 (RXD0)
- new net: R11.2, SW3.2 (B), U1.3 (EN)
- new net: J7.1, U1.37 (TXD0)
Other:
- moved on the sheet: C28, J1, J2, J3, J4, J6, R3, R4, R5, R6, R7, R8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

Commit message: new schematics
Connections:
- net SCL: now also U1.17 (IO9)
- net SDA: now also U1.12 (IO8)
- no-connect marks 4 -> 7
Changed lines of the file:
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@@
+	)
+	(no_connect
+		(at 104.14 92.71)
+	)
+	(no_connect
+		(at 104.14 87.63)
+	)
+	(no_connect
+		(at 104.14 90.17)
 	)
 	(no_connect
@@
 		)
 	)
+	(global_label "SDA"
+		(shape input)
+		(at 73.66 95.25 180)
+		(fields_autoplaced yes)
+		(effects
+			(font
+				(size 1.27 1.27)
+			)
+			(justify right)
+		)
+		(property "Intersheetrefs" "${INTERSHEET_REFS}"
+			(at 67.1067 95.25 0)
+			(hide yes)
+			(show_name no)
+			(do_not_autoplace no)
+			(effects
+				(font
+					(size 1.27 1.27)
+				)
+				(justify right)
+			)
+		)
+	)
 	(global_label "Vibrate"
 		(shape input)
@@
 			(hide yes)
 			(show_name no)
+			(do_not_autoplace no)
+			(effects
+				(font
+					(size 1.27 1.27)
+				)
+				(justify right)
+			)
+		)
+	)
+	(global_label "SCL"
+		(shape input)
+		(at 73.66 97.79 180)
+		(fields_autoplaced yes)
+		(effects
+			(font
+				(size 1.27 1.27)
+			)
+			(justify right)
+		)
+		(property "Intersheetrefs" "${INTERSHEET_REFS}"
+			(at 67.1672 97.79 0)
+			(hide yes)
+			(show_name no)
