File: SmarterWatch_KiCad/Humidity.kicad_sch (KiCad schematic)
At the start: 1 part, among them U6 SHTC3

Commit message: Footprint Stuff
Parts:
- U6: footprint Sensor_Humidity:Sensirion_DFN-4-1EP_2x2mm_P1mm_EP0.7x1.6mm -> (none)
Changed lines of the file:
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@@
 			)
 		)
-		(property "Footprint" "Sensor_Humidity:Sensirion_DFN-4-1EP_2x2mm_P1mm_EP0.7x1.6mm"
+		(property "Footprint" ""
 			(at 135.89 99.06 0)
 			(effects

Commit message: added pad to symbol
Parts:
- U6: footprint (none) -> Custom_Foot:SHTC3_SEN
Changed lines of the file:
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@@
 			)
 		)
-		(property "Footprint" ""
+		(property "Footprint" "Custom_Foot:SHTC3_SEN"
 			(at 135.89 99.06 0)
 			(effects

Commit message: via stuff
Connections:
- net +3.3V_sensor renamed +3.3V
Changed lines of the file:
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@@
-		)
-	)
-	(global_label "+3.3V_sensor"
-		(shape input)
-		(at 133.35 77.47 90)
-		(fields_autoplaced yes)
-		(effects
-			(font
-				(size 1.27 1.27)
-			)
-			(justify left)
-		)
-		(property "Intersheetrefs" "${INTERSHEET_REFS}"
-			(at 133.35 61.6034 90)
-			(effects
-				(font
-					(size 1.27 1.27)
-				)
-				(justify left)
-				(hide yes)
-			)
 		)
 	)
@@
 			)
 		)
+	)
+	(symbol
+		(lib_id "power:+3.3V")
+		(at 133.35 77.47 0)
+		(unit 1)
+		(exclude_from_sim no)
+		(in_bom yes)
+		(on_board yes)
+		(dnp no)
+		(fields_autoplaced yes)
+		(property "Reference" "#PWR032"
+			(at 133.35 81.28 0)
+			(effects
+				(font
+					(size 1.27 1.27)
+				)
+				(hide yes)
+			)
+		)
+		(property "Value" "+3.3V"
+			(at 133.35 72.39 0)
+			(effects
+				(font
+					(size 1.27 1.27)
+				)
+			)
+		)
+		(property "Footprint" ""
+			(at 133.35 77.47 0)
+			(effects
+				(font
+					(size 1.27 1.27)
+				)
+				(hide yes)
+			)
+		)
+		(property "Datasheet" ""
+			(at 133.35 77.47 0)
+			(effects
+				(font
+					(size 1.27 1.27)
+				)
+				(hide yes)
+			)
+		)
+		(property "Description" "Power symbol creates a global label with name \"+3.3V\""
+			(at 133.35 77.47 0)
+			(effects
+				(font
+					(size 1.27 1.27)
+				)
+				(hide yes)
+			)
+		)
+		(pin "1"
+		)
+		(instances
+			(project ""
+				(path "/52181fb0-1be8-41da-83b2-7d5a62778ff4/32cbc301-99d8-4fa0-b16c-40efe0d038ae"
+					(reference "#PWR032")
+					(unit 1)
+				)
+			)
+		)
