File: SmarterWatch_KiCad/LDO.kicad_sch (KiCad schematic)
At the start: 2 parts, among them U4 TCR2EE10

Commit message: Footprint Stuff
Parts:
- U4: footprint Package_TO_SOT_SMD:SOT-553 -> (none)
Changed lines of the file:
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@@
 			)
 		)
-		(property "Footprint" "Package_TO_SOT_SMD:SOT-553"
+		(property "Footprint" ""
 			(at 149.86 107.95 0)
 			(effects

Commit message: Jumper Footprint
Parts:
- U4: footprint (none) -> Custom_Foot:SOT-25 SMV_TOS
Changed lines of the file:
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@@
 			)
 		)
-		(property "Footprint" ""
+		(property "Footprint" "Custom_Foot:SOT-25   SMV_TOS"
 			(at 149.86 107.95 0)
 			(effects
