File: SmarterWatch_KiCad/Light Sensor.kicad_sch (KiCad schematic)
At the start: 2 parts, among them U2 TSL25911FN

Commit message: Footprint Stuff
Parts:
- U2: footprint OptoDevice:AMS_TSL25911FN -> TerminalBlock_CUI:SON-06-FN_2000X2400_AMS
Changed lines of the file:
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@@
 			)
 		)
-		(property "Footprint" "OptoDevice:AMS_TSL25911FN"
+		(property "Footprint" "TerminalBlock_CUI:SON-06-FN_2000X2400_AMS"
 			(at 129.54 100.33 0)
 			(effects

Commit message: YOUR MOM!
YOUR MOM! YOUR MOM! YOUR MOM! YOUR MOM! YOUR MOM! YOUR MOM! YOUR MOM! YOUR MOM! YOUR MOM! YOUR MOM! YOUR MOM! YOUR MOM! YOUR MOM! YOUR MOM! YOUR MOM! YOUR MOM! YOUR MOM! YOUR MOM! YOUR MOM!
Parts:
- U2: footprint TerminalBlock_CUI:SON-06-FN_2000X2400_AMS -> Custom_Foot:SON-06-FN_2000X2400_AMS-L
Changed lines of the file:
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@@
 			)
 		)
-		(property "Footprint" "TerminalBlock_CUI:SON-06-FN_2000X2400_AMS"
+		(property "Footprint" "Custom_Foot:SON-06-FN_2000X2400_AMS-L"
 			(at 129.54 100.33 0)
 			(effects

Commit message: via stuff
Connections:
- net +3.3V_sensor renamed +3.3V
Changed lines of the file:
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@@
-		)
-	)
-	(global_label "+3.3V_sensor"
-		(shape input)
-		(at 161.29 77.47 0)
-		(fields_autoplaced yes)
-		(effects
-			(font
-				(size 1.27 1.27)
-			)
-			(justify left)
-		)
-		(property "Intersheetrefs" "${INTERSHEET_REFS}"
-			(at 177.1566 77.47 0)
-			(effects
-				(font
-					(size 1.27 1.27)
-				)
-				(justify left)
-				(hide yes)
-			)
 		)
 	)
@@
 			)
 		)
+	)
+	(symbol
+		(lib_id "power:+3.3V")
+		(at 161.29 77.47 0)
+		(unit 1)
+		(exclude_from_sim no)
+		(in_bom yes)
+		(on_board yes)
+		(dnp no)
+		(fields_autoplaced yes)
+		(property "Reference" "#PWR031"
+			(at 161.29 81.28 0)
+			(effects
+				(font
+					(size 1.27 1.27)
+				)
+				(hide yes)
+			)
+		)
+		(property "Value" "+3.3V"
+			(at 161.29 72.39 0)
+			(effects
+				(font
+					(size 1.27 1.27)
+				)
+			)
+		)
+		(property "Footprint" ""
+			(at 161.29 77.47 0)
+			(effects
+				(font
+					(size 1.27 1.27)
+				)
+				(hide yes)
+			)
+		)
+		(property "Datasheet" ""
+			(at 161.29 77.47 0)
+			(effects
+				(font
+					(size 1.27 1.27)
+				)
+				(hide yes)
+			)
+		)
+		(property "Description" "Power symbol creates a global label with name \"+3.3V\""
+			(at 161.29 77.47 0)
+			(effects
+				(font
+					(size 1.27 1.27)
+				)
+				(hide yes)
+			)
+		)
+		(pin "1"
+		)
+		(instances
+			(project ""
+				(path "/52181fb0-1be8-41da-83b2-7d5a62778ff4/ff37529c-7f13-4764-a7bc-f886fcded995"
+					(reference "#PWR031")
+					(unit 1)
+				)
+			)
+		)
