File: SmarterWatch_KiCad/MOSFET.kicad_sch (KiCad schematic)
At the start: 3 parts, among them Q1 2N7002

Commit message: Yay!
Parts:
- removed Q1: 2N7002, Package_TO_SOT_SMD:SOT-23, symbol dk_Transistors-FETs-MOSFETs-Single:2N7002
- removed R10: 1k, Resistor_SMD:R_0402_1005Metric, symbol Device:R
- removed R11: 10k, Resistor_SMD:R_0402_1005Metric, symbol Device:R
