File: SmarterWatch_KiCad/Screen.kicad_sch (KiCad schematic)
At the start: 7 parts, among them Q2 2N7002, Q3 2N7002

Commit message: Footprint Stuff
Parts:
- U8: footprint Connector_PinSocket_2.54mm:PinSocket_1x08_P2.54mm_Vertical -> (none)
Changed lines of the file:
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@@
 			)
 		)
-		(property "Footprint" "Connector_PinSocket_2.54mm:PinSocket_1x08_P2.54mm_Vertical"
+		(property "Footprint" ""
 			(at 130.81 90.17 0)
 			(effects

Commit message: named screen
Parts:
- U8: value ~ -> ST7735
Changed lines of the file:
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@@
 			)
 		)
-		(property "Value" "~"
+		(property "Value" "ST7735"
 			(at 140.97 101.5999 0)
 			(effects

Commit message: footprint
Parts:
- U8: footprint (none) -> Connector_PinSocket_2.54mm:PinSocket_1x08_P2.54mm_Vertical
Changed lines of the file:
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@@
 			)
 		)
-		(property "Footprint" ""
+		(property "Footprint" "Connector_PinSocket_2.54mm:PinSocket_1x08_P2.54mm_Vertical"
 			(at 130.81 90.17 0)
 			(effects
