File: SmarterWatch_KiCad/Screen.kicad_sch (KiCad schematic)
At the start: 7 parts, among them Q2 2N7002, Q3 2N7002, U8 ST7735

Commit message: new schematics
Parts:
- removed Q2, Q3: 2N7002, Package_TO_SOT_SMD:SOT-23, symbol dk_Transistors-FETs-MOSFETs-Single:2N7002
- removed R13: 1k, Resistor_SMD:R_0402_1005Metric, symbol Device:R
- removed R15: 10k, Resistor_SMD:R_0402_1005Metric, symbol Device:R
- added J10: Conn_01x07_Pin, symbol Connector:Conn_01x07_Pin
Connections:
- net +3.3V: now also R12.2, R14.2, U8.8 (VCC), J10.1 (Pin_1)
- net GND: now also J10.2 (Pin_2)
- net MOSI: now also J10.3 (Pin_3)
- net SCLK: now also J10.4 (Pin_4)
- net Screen_A0: now also J10.6 (Pin_6)
- net Screen_CS: now also J10.5 (Pin_5)
- net Screen_Reset: now also J10.7 (Pin_7)
Other:
- moved on the sheet: R12, R14
