File: SmarterWatch_KiCad/USBC.kicad_sch (KiCad schematic)
At the start: 1 part, among them J3 CX70M-24P1

Commit message: checking sum schematic and touching the wires together forever
Parts:
- added R24, R25: 33k, Resistor_SMD:R_0402_1005Metric, symbol Device:R
Connections:
- net GND: now also R24.2, R25.1
- net at J3.A5: now also R24.1
- net at J3.B5: now also R25.2
- no-connect marks 12 -> 10

Commit message: Minor Changes
Parts:
- renumbered J3 to J5, R25 to R16, R24 to R17
Changed lines of the file:
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@@
 		(dnp no)
 		(fields_autoplaced yes)
-		(property "Reference" "#PWR052"
+		(property "Reference" "#PWR056"
 			(at 132.08 92.71 0)
 			(effects
@@
 			(project "Smarter Watch Stuff"
 				(path "/52181fb0-1be8-41da-83b2-7d5a62778ff4/cfac10be-be17-4cdb-a849-9d1c07b85e1a"
-					(reference "#PWR052")
+					(reference "#PWR056")
 					(unit 1)
 				)
@@
 		(dnp no)
 		(fields_autoplaced yes)
-		(property "Reference" "#PWR054"
+		(property "Reference" "#PWR058"
 			(at 135.89 116.84 0)
 			(effects
@@
 			(project "Smarter Watch Stuff"
 				(path "/52181fb0-1be8-41da-83b2-7d5a62778ff4/cfac10be-be17-4cdb-a849-9d1c07b85e1a"
-					(reference "#PWR054")
+					(reference "#PWR058")
 					(unit 1)
 				)
@@
 		(dnp no)
 		(fields_autoplaced yes)
-		(property "Reference" "#PWR056"
+		(property "Reference" "#PWR060"
 			(at 149.86 80.01 0)
 			(effects
@@
 			(project "Smarter Watch Stuff"
 				(path "/52181fb0-1be8-41da-83b2-7d5a62778ff4/cfac10be-be17-4cdb-a849-9d1c07b85e1a"
-					(reference "#PWR056")
+					(reference "#PWR060")
 					(unit 1)
 				)
@@
 		(dnp no)
 		(fields_autoplaced yes)
-		(property "Reference" "#PWR058"
+		(property "Reference" "#PWR062"
 			(at 160.02 100.33 0)
 			(effects
@@
 			(project "Smarter Watch Stuff"
 				(path "/52181fb0-1be8-41da-83b2-7d5a62778ff4/cfac10be-be17-4cdb-a849-9d1c07b85e1a"
-					(reference "#PWR058")
+					(reference "#PWR062")
 					(unit 1)
 				)
@@
 		(dnp no)
 		(fields_autoplaced yes)
-		(property "Reference" "R24"
+		(property "Reference" "R17"
 			(at 157.48 76.2 90)
 			(effects
@@
 			(project ""
 				(path "/52181fb0-1be8-41da-83b2-7d5a62778ff4/cfac10be-be17-4cdb-a849-9d1c07b85e1a"
-					(reference "R24")
+					(reference "R17")
 					(unit 1)
 				)
@@
 		(dnp no)
 		(fields_autoplaced yes)
-		(property "Reference" "#PWR051"
+		(property "Reference" "#PWR055"
 			(at 132.08 80.01 0)
 			(effects
@@
 			(project ""
 				(path "/52181fb0-1be8-41da-83b2-7d5a62778ff4/cfac10be-be17-4cdb-a849-9d1c07b85e1a"
-					(reference "#PWR051")
+					(reference "#PWR055")
 					(unit 1)
 				)
@@
 		(dnp no)
 		(fields_autoplaced yes)
-		(property "Reference" "#PWR057"
+		(property "Reference" "#PWR061"
 			(at 149.86 92.71 0)
 			(effects
@@
 			(project "Smarter Watch Stuff"
 				(path "/52181fb0-1be8-41da-83b2-7d5a62778ff4/cfac10be-be17-4cdb-a849-9d1c07b85e1a"
-					(reference "#PWR057")
+					(reference "#PWR061")
 					(unit 1)
 				)
@@
 		(dnp no)
 		(fields_autoplaced yes)
-		(property "Reference" "#PWR068"
+		(property "Reference" "#PWR063"
 			(at 167.64 82.55 0)
 			(effects
@@
 			(project ""
 				(path "/52181fb0-1be8-41da-83b2-7d5a62778ff4/cfac10be-be17-4cdb-a849-9d1c07b85e1a"
-					(reference "#PWR068")
+					(reference "#PWR063")
 					(unit 1)
 				)
@@
 		(dnp no)
 		(fields_autoplaced yes)
-		(property "Reference" "R25"
+		(property "Reference" "R16"
 			(at 124.46 83.82 90)
 			(effects
@@
 			(project "Smarter Watch Stuff"
 				(path "/52181fb0-1be8-41da-83b2-7d5a62778ff4/cfac10be-be17-4cdb-a849-9d1c07b85e1a"
-					(reference "R25")
+					(reference "R16")
 					(unit 1)
 				)
@@
 		(dnp no)
 		(fields_autoplaced yes)
-		(property "Reference" "#PWR053"
+		(property "Reference" "#PWR057"
 			(at 121.92 100.33 0)
 			(effects
@@
 			(project ""
 				(path "/52181fb0-1be8-41da-83b2-7d5a62778ff4/cfac10be-be17-4cdb-a849-9d1c07b85e1a"
-					(reference "#PWR053")
+					(reference "#PWR057")
 					(unit 1)
 				)
@@
 		(dnp no)
 		(fields_autoplaced yes)
-		(property "Reference" "#PWR069"
+		(property "Reference" "#PWR053"
 			(at 114.3 90.17 0)
 			(effects
@@
 			(project "Smarter Watch Stuff"
 				(path "/52181fb0-1be8-41da-83b2-7d5a62778ff4/cfac10be-be17-4cdb-a849-9d1c07b85e1a"
-					(reference "#PWR069")
+					(reference "#PWR053")
 					(unit 1)
 				)
@@
 		(dnp no)
 		(fields_autoplaced yes)
-		(property "Reference" "#PWR055"
+		(property "Reference" "#PWR059"
 			(at 160.02 72.39 0)
 			(effects
@@
 			(project "Smarter Watch Stuff"
 				(path "/52181fb0-1be8-41da-83b2-7d5a62778ff4/cfac10be-be17-4cdb-a849-9d1c07b85e1a"
-					(reference "#PWR055")
+					(reference "#PWR059")
 					(unit 1)
 				)
@@
 		(dnp no)
 		(fields_autoplaced yes)
-		(property "Reference" "#PWR050"
+		(property "Reference" "#PWR054"
 			(at 121.92 72.39 0)
 			(effects
@@
 			(project "Smarter Watch Stuff"
 				(path "/52181fb0-1be8-41da-83b2-7d5a62778ff4/cfac10be-be17-4cdb-a849-9d1c07b85e1a"
-					(reference "#PWR050")
+					(reference "#PWR054")
 					(unit 1)
 				)
@@
 		(dnp no)
 		(fields_autoplaced yes)
-		(property "Reference" "J3"
+		(property "Reference" "J5"
 			(at 140.97 59.69 0)
 			(effects
@@
 			(project "Smarter Watch Stuff"
 				(path "/52181fb0-1be8-41da-83b2-7d5a62778ff4/cfac10be-be17-4cdb-a849-9d1c07b85e1a"
-					(reference "J3")
-					(unit 1)
-				)
+					(reference "J5")
+					(unit 1)
+				)

Commit message: more prgrs
Parts:
- added FB1, FB2: FerriteBead, Resistor_SMD:R_0402_1005Metric, symbol Device:FerriteBead
Connections:
- net GND: now also FB1.2; no longer J5.SH
- new net: FB1.1, FB2.1, J5.S1
Changed lines of the file:
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@@
 	(generator_version "9.0")
 	(paper "A4")
+	(junction
+		(at 135.89 111.76)
+		(diameter 0)
+		(color 0 0 0 0)
+	)
 	(no_connect
 		(at 128.27 97.79)
@@
 	(no_connect
 		(at 128.27 95.25)
+	)
+	(wire
+		(pts
+			(xy 128.27 111.76) (xy 135.89 111.76)
+		)
+		(stroke
+			(width 0)
+			(type default)
+		)
+	)
+	(wire
+		(pts
+			(xy 135.89 111.76) (xy 135.89 110.49)
+		)
+		(stroke
+			(width 0)
+			(type default)
+		)
+	)
+	(wire
+		(pts
+			(xy 135.89 119.38) (xy 135.89 120.65)
+		)
+		(stroke
+			(width 0)
+			(type default)
+		)
 	)
 	(global_label "USB_D+"
@@
 	(symbol
 		(lib_id "power:GND")
-		(at 135.89 110.49 0)
+		(at 135.89 120.65 0)
 		(unit 1)
 		(exclude_from_sim no)
@@
 		(fields_autoplaced yes)
 		(property "Reference" "#PWR058"
-			(at 135.89 116.84 0)
+			(at 135.89 127 0)
 			(effects
 				(font
@@
 		)
 		(property "Value" "GND"
-			(at 135.89 115.57 0)
+			(at 135.89 125.73 0)
 			(effects
 				(font
@@
 		)
 		(property "Footprint" ""
-			(at 135.89 110.49 0)
+			(at 135.89 120.65 0)
 			(effects
 				(font
@@
 		)
 		(property "Datasheet" ""
-			(at 135.89 110.49 0)
+			(at 135.89 120.65 0)
 			(effects
 				(font
@@
 		)
 		(property "Description" "Power symbol creates a global label with name \"GND\" , ground"
-			(at 135.89 110.49 0)
+			(at 135.89 120.65 0)
 			(effects
 				(font
@@
 	)
 	(symbol
+		(lib_id "Device:FerriteBead")
+		(at 128.27 115.57 0)
+		(unit 1)
+		(exclude_from_sim no)
+		(in_bom yes)
+		(on_board yes)
+		(dnp no)
+		(fields_autoplaced yes)
+		(property "Reference" "FB2"
+			(at 132.08 114.2491 0)
+			(effects
+				(font
+					(size 1.27 1.27)
+				)
+				(justify left)
+			)
+		)
+		(property "Value" "FerriteBead"
+			(at 132.08 116.7891 0)
+			(effects
+				(font
+					(size 1.27 1.27)
+				)
+				(justify left)
+			)
+		)
+		(property "Footprint" "Resistor_SMD:R_0402_1005Metric"
+			(at 126.492 115.57 90)
+			(effects
+				(font
+					(size 1.27 1.27)
+				)
+				(hide yes)
+			)
+		)
+		(property "Datasheet" "~"
+			(at 128.27 115.57 0)
+			(effects
+				(font
+					(size 1.27 1.27)
+				)
+				(hide yes)
+			)
+		)
+		(property "Description" "Ferrite bead"
+			(at 128.27 115.57 0)
+			(effects
+				(font
+					(size 1.27 1.27)
+				)
+				(hide yes)
+			)
+		)
+		(pin "1"
+		)
+		(pin "2"
+		)
+		(instances
+			(project "Smarter Watch Stuff"
+				(path "/52181fb0-1be8-41da-83b2-7d5a62778ff4/cfac10be-be17-4cdb-a849-9d1c07b85e1a"
+					(reference "FB2")
+					(unit 1)
+				)
+			)
+		)
+	)
+	(symbol
 		(lib_id "Device:R")
 		(at 124.46 90.17 90)
@@
 	)
 	(symbol
+		(lib_id "Device:FerriteBead")
+		(at 135.89 115.57 0)
+		(unit 1)
+		(exclude_from_sim no)
+		(in_bom yes)
+		(on_board yes)
+		(dnp no)
+		(fields_autoplaced yes)
+		(property "Reference" "FB1"
+			(at 139.7 114.2491 0)
+			(effects
+				(font
+					(size 1.27 1.27)
+				)
+				(justify left)
+			)
+		)
+		(property "Value" "FerriteBead"
+			(at 139.7 116.7891 0)
+			(effects
+				(font
+					(size 1.27 1.27)
+				)
+				(justify left)
+			)
+		)
+		(property "Footprint" "Resistor_SMD:R_0402_1005Metric"
+			(at 134.112 115.57 90)
+			(effects
+				(font
+					(size 1.27 1.27)
+				)
+				(hide yes)
+			)
+		)
+		(property "Datasheet" "~"
+			(at 135.89 115.57 0)
+			(effects
+				(font
+					(size 1.27 1.27)
+				)
+				(hide yes)
+			)
+		)
+		(property "Description" "Ferrite bead"
+			(at 135.89 115.57 0)
+			(effects
+				(font
+					(size 1.27 1.27)
+				)
+				(hide yes)
+			)
+		)
+		(pin "1"
+		)
+		(pin "2"
+		)
+		(instances
+			(project ""
+				(path "/52181fb0-1be8-41da-83b2-7d5a62778ff4/cfac10be-be17-4cdb-a849-9d1c07b85e1a"
+					(reference "FB1")
+					(unit 1)
+				)
+			)
+		)
+	)
+	(symbol
 		(lib_id "power:GND")
 		(at 128.27 100.33 270)
@@
 		(pin "A2"
 		)
-		(pin "SH"
+		(pin "S1"
 		)
 		(pin "A3"

Commit message: FINAL
Connections:
- net GND: now also FB2.2
