File: SmarterWatch_KiCad/Smarter Watch Stuff.kicad_sch (KiCad schematic)
At the start: 0 parts

Commit message: Added Heart Symbol
Other:
- added sheet New Heart (NewHeart.kicad_sch)
Changed lines of the file:
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@@
+	)
+	(sheet
+		(at 187.96 20.32)
+		(size 36.195 24.13)
+		(exclude_from_sim no)
+		(in_bom yes)
+		(on_board yes)
+		(dnp no)
+		(fields_autoplaced yes)
+		(stroke
+			(width 0.1524)
+			(type solid)
+		)
+		(fill
+			(color 0 0 0 0)
+		)
+		(property "Sheetname" "New Heart"
+			(at 187.96 19.6084 0)
+			(show_name no)
+			(do_not_autoplace no)
+			(effects
+				(font
+					(size 1.27 1.27)
+				)
+				(justify left bottom)
+			)
+		)
+		(property "Sheetfile" "NewHeart.kicad_sch"
+			(at 187.96 45.0346 0)
+			(show_name no)
+			(do_not_autoplace no)
+			(effects
+				(font
+					(size 1.27 1.27)
+				)
+				(justify left top)
+			)
+		)
+		(instances
+			(project "Smarter Watch Stuff"
+				(path "/52181fb0-1be8-41da-83b2-7d5a62778ff4"
+					(page "24")
+				)
+			)
+		)
 	)
 	(sheet

Commit message: update
Other:
- removed sheet Clock
Changed lines of the file:
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@@
-	)
-	(sheet
-		(at 13.97 160.02)
-		(size 36.83 38.1)
-		(exclude_from_sim no)
-		(in_bom yes)
-		(on_board yes)
-		(dnp no)
-		(fields_autoplaced yes)
-		(stroke
-			(width 0.1524)
-			(type solid)
-		)
-		(fill
-			(color 0 0 0 0)
-		)
-		(property "Sheetname" "Clock"
-			(at 13.97 159.3084 0)
-			(show_name no)
-			(do_not_autoplace no)
-			(effects
-				(font
-					(size 1.27 1.27)
-				)
-				(justify left bottom)
-			)
-		)
-		(property "Sheetfile" "untitled.kicad_sch"
-			(at 13.97 198.7046 0)
-			(show_name no)
-			(do_not_autoplace no)
-			(effects
-				(font
-					(size 1.27 1.27)
-				)
-				(justify left top)
-			)
-		)
-		(instances
-			(project "Smarter Watch Stuff"
-				(path "/52181fb0-1be8-41da-83b2-7d5a62778ff4"
-					(page "2")
-				)
-			)
-		)
 	)
 	(sheet
